Commit message: feat: 修改了xacro中的问题

File: lite3_description/xacro/const.xacro (robot description, xacro)
@@ -31,3 +31,14 @@
   <xacro:property name="foot_mass" value="0.08179029876178574"/>
   <xacro:property name="foot_radius" value="0.013"/>
+  <!-- shank -->
+  <xacro:property name="shank_mass" value="0.1567647392934227"/>
+  <xacro:property name="shank_com_x" value="0.00585"/>
+  <xacro:property name="shank_com_y" value="-8.732e-07"/>
+  <xacro:property name="shank_com_z" value="-0.12"/>
+  <xacro:property name="shank_ixx" value="9.104550629239001e-04"/>
+  <xacro:property name="shank_ixy" value="-1.690647476476001e-08"/>
+  <xacro:property name="shank_ixz" value="9.41971624706656e-06"/>
+  <xacro:property name="shank_iyy" value="9.353157488964166e-04"/>
+  <xacro:property name="shank_iyz" value="7.70211998592336e-09"/>
+  <xacro:property name="shank_izz" value="4.30081045672405e-05"/>
 </robot>

File: lite3_description/xacro/leg.xacro (robot description, xacro)
@@ -24,5 +24,4 @@
     <link name="${name}_HIP">
       <inertial>
-        <inertia ixx="0.00014538" ixy="8.1579E-07" ixz="-1.264E-05" iyy="0.00024024" iyz="1.3443E-06" izz="0.00013038"/>
         <origin xyz="${hip_com_x*front_hind} ${hip_com_y*mirror} ${hip_com_z}"/>
         <mass value="${hip_mass}"/>
@@ -55,5 +54,4 @@
             iyy="${thigh_iyy}" iyz="${thigh_iyz*mirror}"
             izz="${thigh_izz}"/>
-        <inertia ixx="0.001" ixy="-2.5E-06" ixz="-1.12E-04" iyy="0.00116" iyz="3.75E-07" izz="2.68E-04"/>
       </inertial>
       <visual>
@@ -85,7 +83,10 @@
     <link name="${name}_SHANK">
       <inertial>
-        <origin xyz="0.00585 -8.732E-07 -0.12"/>
-        <mass value="0.1567647392934227"></mass>
-        <inertia ixx="9.104550629239001e-04" ixy="-1.690647476476001e-08" ixz="9.41971624706656e-06" iyy="9.353157488964166e-04" iyz="7.70211998592336e-09" izz="4.30081045672405e-05"/>
+        <origin xyz="${shank_com_x} ${shank_com_y*mirror} ${shank_com_z}"/>
+        <mass value="${shank_mass}"/>
+        <inertia
+            ixx="${shank_ixx}" ixy="${shank_ixy*mirror}" ixz="${shank_ixz}"
+            iyy="${shank_iyy}" iyz="${shank_iyz*mirror}"
+            izz="${shank_izz}"/>
       </inertial>
       <visual>
@@ -121,27 +122,4 @@
       </collision>
     </link>
-    <gazebo reference="${name}_HIP">
-      <mu1>0.2</mu1>
-      <mu2>0.2</mu2>
-    </gazebo>
-    <gazebo reference="${name}_THIGH">
-      <mu1>0.2</mu1>
-      <mu2>0.2</mu2>
-      <self_collide>0</self_collide>
-      <kp value="1000000.0"/>
-      <kd value="100.0"/>
-    </gazebo>
-    <gazebo reference="${name}_SHANK">
-      <mu1>0.6</mu1>
-      <mu2>0.6</mu2>
-      <self_collide>1</self_collide>
-    </gazebo>
-    <gazebo reference="${name}_FOOT">
-      <mu1>0.6</mu1>
-      <mu2>0.6</mu2>
-      <self_collide>1</self_collide>
-      <kp value="1000000.0"/>
-      <kd value="100.0"/>
-    </gazebo>
     <xacro:leg_transmission name="${name}"/>
   </xacro:macro>

File: lite3_description/xacro/transmission.xacro (robot description, xacro)
@@ -11,19 +11,19 @@
       </actuator>
     </transmission>
-    <transmission name="{name}_HipY_tran">
+    <transmission name="${name}_HipY_tran">
       <type>transmission_interface/SimpleTransmission</type>
-      <joint name="{name}_HipY">
+      <joint name="${name}_HipY">
         <hardwareInterface>hardware_interface/EffortJointInterface</hardwareInterface>
       </joint>
-      <actuator name="{name}_HipY_motor">
+      <actuator name="${name}_HipY_motor">
         <mechanicalReduction>1</mechanicalReduction>
       </actuator>
     </transmission>
-    <transmission name="{name}_Knee_tran">
+    <transmission name="${name}_Knee_tran">
       <type>transmission_interface/SimpleTransmission</type>
-      <joint name="{name}_Knee">
+      <joint name="${name}_Knee">
         <hardwareInterface>hardware_interface/EffortJointInterface</hardwareInterface>
       </joint>
-      <actuator name="{name}_Knee_motor">
+      <actuator name="${name}_Knee_motor">
         <mechanicalReduction>1</mechanicalReduction>
       </actuator>

Commit message: feat: 新增reamde描述

File: lite3_description/xacro/const.xacro (robot description, xacro)
@@ -29,5 +29,5 @@
   <xacro:property name="thigh_izz" value="2.68E-04"/>
   <!-- foot -->
-  <xacro:property name="foot_mass" value="0.08179029876178574"/>
+  <xacro:property name="foot_mass" value="0.01519029876178574"/>
   <xacro:property name="foot_radius" value="0.013"/>
   <!-- shank -->
