Commit message: feat: 适配 Realsense D435i 相机并优化文档
主要改动：
1. Realsense D435i 相机适配
   - 简化为仅 RGB 模式（用于 FAST-LIVO 雷达点着色）
   - 使用标准 libgazebo_ros_camera.so 插件
   - 移除深度和红外相机配置

2. Livox Mid-360 TF 优化
   - 将静态 TF 从 launch 文件移动到 URDF 模型
   - 添加 mid360_livox_laser frame 到 URDF
   - 统一 TF 管理方式

3. 删除 realsense_gazebo_plugin 子模块
   - 不再使用 realsense_gazebo_plugin
   - 使用 Gazebo 标准相机插件替代

4. 文档整理
   - 新增 sensor_configuration.md - 传感器配置文档
   - 新增 keyboard_control_guide.md - 键盘控制指南
   - 新增 troubleshooting.md - 故障排除指南
   - 新增 docs/README.md - 文档索引
   - 精简主 README，移除不相关内容到 docs

5. 代码修正
   - 修正 launch 文件中的注释
   - 明确 GAZEBO_PLUGIN_PATH 设置说明

File: lite3_description/xacro/sensors/d435i_sensor.xacro (robot description, xacro)
@@ -2,8 +2,12 @@
 <robot xmlns:xacro="http://ros.org/wiki/xacro">
   <xacro:property name="M_PI" value="3.1415926535897931"/>
+  <!--
+    Realsense D435i 相机传感器配置（仅 RGB，用于 FAST-LIVO 雷达点着色）
+    仅发布 RGB 图像和 CameraInfo，不需要深度和红外数据
+  -->
   <xacro:macro name="d435i_sensor" params="name:=d435i parent:=base_link
                                           xyz:='0 0 0' rpy:='0 0 0'
                                           topic_ns:=camera visualize:=false">
-    <!-- 实体 Link -->
+    <!-- 物理 Link（相机实体） -->
     <link name="${name}_link">
       <inertial>
@@ -12,16 +16,21 @@
       </inertial>
       <visual>
-        <geometry><box size="0.025 0.090 0.025"/></geometry>
-        <material name="${name}_material"><color rgba="0.1 0.1 0.1 1.0"/></material>
+        <origin xyz="0 0 0" rpy="0 0 0"/>
+        <geometry>
+          <box size="0.025 0.090 0.025"/>
+        </geometry>
+        <material name="${name}_material">
+          <color rgba="0.1 0.1 0.1 1.0"/>
+        </material>
       </visual>
       <collision>
-        <geometry><box size="0.025 0.090 0.025"/></geometry>
+        <geometry>
+          <box size="0.025 0.090 0.025"/>
+        </geometry>
       </collision>
     </link>
-    <!-- 光学 Frames -->
+    <!-- 仅保留 color_optical_frame（用于 RGB 相机光学坐标系） -->
     <link name="${name}_color_optical_frame"/>
-    <link name="${name}_depth_optical_frame"/>
-    <link name="${name}_infra1_optical_frame"/>
-    <link name="${name}_infra2_optical_frame"/>
+    <!-- 安装到机器人的 Joint -->
     <joint name="${name}_joint" type="fixed">
       <parent link="${parent}"/>
@@ -29,9 +38,6 @@
       <origin xyz="${xyz}" rpy="${rpy}"/>
     </joint>
-    <joint name="${name}_depth_optical_joint" type="fixed">
-      <parent link="${name}_link"/>
-      <child link="${name}_depth_optical_frame"/>
-      <origin xyz="0.005 0 0" rpy="${-M_PI/2} 0 ${-M_PI/2}"/>
-    </joint>
+    <!-- color_optical_frame 相对于 link 的偏移（RV 坐标系到光学坐标系） -->
+    <!-- D435i 彩色相机光心相对于 IMU 的偏移：X=5mm, Y=17.5mm, Z=0mm -->
     <joint name="${name}_color_optical_joint" type="fixed">
       <parent link="${name}_link"/>
@@ -39,56 +45,34 @@
       <origin xyz="0.005 0.0175 0" rpy="${-M_PI/2} 0 ${-M_PI/2}"/>
     </joint>
-    <joint name="${name}_infra1_optical_joint" type="fixed">
-      <parent link="${name}_link"/>
-      <child link="${name}_infra1_optical_frame"/>
-      <origin xyz="0.005 -0.0175 0" rpy="${-M_PI/2} 0 ${-M_PI/2}"/>
-    </joint>
-    <joint name="${name}_infra2_optical_joint" type="fixed">
-      <parent link="${name}_link"/>
-      <child link="${name}_infra2_optical_frame"/>
-      <origin xyz="0.005 -0.055 0" rpy="${-M_PI/2} 0 ${-M_PI/2}"/>
-    </joint>
-    <!-- Gazebo 插件 -->
+    <!-- Gazebo 传感器：仅 RGB 相机（用于 FAST-LIVO 着色） -->
     <gazebo reference="${name}_link">
-      <sensor type="depth" name="${name}_depth">
+      <sensor type="camera" name="${name}_color">
         <camera>
-          <horizontal_fov>1.211</horizontal_fov>
-          <image><width>1280</width><height>720</height></image>
-          <clip><near>0.1</near><far>10.0</far></clip>
+          <!-- D435i RGB 相机参数 -->
+          <horizontal_fov>1.211</horizontal_fov>  <!-- 87° 水平视场角 -->
+          <image>
+            <width>1280</width>
+            <height>720</height>
+            <format>R8G8B8</format>
+          </image>
+          <clip>
+            <near>0.1</near>
+            <far>10.0</far>
+          </clip>
         </camera>
         <always_on>1</always_on>
-        <update_rate>30</update_rate>
+        <update_rate>30.0</update_rate>
         <visualize>${visualize}</visualize>
+        <!-- 使用标准 ROS2 相机插件（稳定可靠） -->
+        <plugin name="${name}_color_plugin" filename="libgazebo_ros_camera.so">
+          <ros>
+            <namespace>/${topic_ns}</namespace>
+            <remapping>image_raw:=color/image_raw</remapping>
+            <remapping>camera_info:=color/camera_info</remapping>
+          </ros>
+          <camera_name>color</camera_name>
+          <frame_name>${name}_color_optical_frame</frame_name>
+        </plugin>
       </sensor>
-      <sensor type="camera" name="${name}_color">
-        <camera>
-          <horizontal_fov>1.211</horizontal_fov>
-          <image><width>1280</width><height>720</height><format>R8G8B8</format></image>
-          <clip><near>0.1</near><far>10.0</far></clip>
-        </camera>
-        <always_on>1</always_on>
-        <update_rate>30</update_rate>
-        <visualize>${visualize}</visualize>
-      </sensor>
-      <!-- 使用标准 ROS 插件代替 realsense_gazebo_plugin -->
-      <plugin name="${name}_depth_plugin" filename="libgazebo_ros_depth_camera.so">
-        <ros>
-          <namespace>/${topic_ns}</namespace>
-          <remapping>image_raw:=depth/image_rect_raw</remapping>
-          <remapping>camera_info:=depth/camera_info</remapping>
-          <remapping>points:=depth/color/points</remapping>
-        </ros>
-        <camera_name>depth</camera_name>
-        <frame_name>${name}_depth_optical_frame</frame_name>
-      </plugin>
-      <plugin name="${name}_color_plugin" filename="libgazebo_ros_camera.so">
-        <ros>
-          <namespace>/${topic_ns}</namespace>
-          <remapping>image_raw:=color/image_raw</remapping>
-          <remapping>camera_info:=color/camera_info</remapping>
-        </ros>
-        <camera_name>color</camera_name>
-        <frame_name>${name}_color_optical_frame</frame_name>
-      </plugin>
     </gazebo>
   </xacro:macro>

File: lite3_description/xacro/sensors/mid360_sensor.xacro (robot description, xacro)
@@ -35,4 +35,6 @@
       </inertial>
     </link>
+    <!-- Livox 插件发布的 frame_id 是 mid360_livox_laser，需要添加这个 frame -->
+    <link name="${name}_livox_laser"/>
     <!-- 关键：底座到光学中心的偏移（Livox 官方数据） -->
     <joint name="${name}_base_joint" type="fixed">
@@ -40,4 +42,10 @@
       <child link="${name}_link"/>
       <origin xyz="-0.012 0.0 0.047" rpy="0 0 0"/>
+    </joint>
+    <!-- 添加 mid360_link 到 mid360_livox_laser 的静态 TF（零变换） -->
+    <joint name="${name}_livox_laser_joint" type="fixed">
+      <parent link="${name}_link"/>
+      <child link="${name}_livox_laser"/>
+      <origin xyz="0 0 0" rpy="0 0 0"/>
     </joint>
     <!-- 安装到机器人 -->
